File: noah.sch (KiCad schematic (older format))
At the start: 139 parts, among them U1 ATmega32U4-AU, U2 SRV05-4

Commit message: add LCSC BOM and placing files
Parts:
- D1, D10, D11, D12, D13, D14, D15, D17, D18, D19, D2, D20, D21, D22, D23, D24, D25, D26, D27, D28, D29, D3, D30, D32, D33, D35, D36, D4, D5, D6, D7, D8, D9: LCSC (none) -> C2500
- D16, D31, D34: LCSC (none) -> C81598
Changed lines of the file:
@@
 F 2 "custom_parts:D_SOT-23_ANK" V 7200 2900 50  0001 C CNN
 F 3 "~" V 7200 2900 50  0001 C CNN
+F 4 "C2500" H 7200 2900 50  0001 C CNN "LCSC"
 	1    7200 2900
 	0    -1   -1   0
@@
 F 2 "custom_parts:D_SOT-23_ANK" V 8100 2900 50  0001 C CNN
 F 3 "~" V 8100 2900 50  0001 C CNN
+F 4 "C2500" H 8100 2900 50  0001 C CNN "LCSC"
 	1    8100 2900
 	0    -1   -1   0
@@
 F 2 "custom_parts:D_SOT-23_ANK" V 9000 2900 50  0001 C CNN
 F 3 "~" V 9000 2900 50  0001 C CNN
+F 4 "C2500" H 9000 2900 50  0001 C CNN "LCSC"
 	1    9000 2900
 	0    -1   -1   0
@@
 F 2 "custom_parts:D_SOT-23_ANK" V 9900 2900 50  0001 C CNN
 F 3 "~" V 9900 2900 50  0001 C CNN
+F 4 "C2500" H 9900 2900 50  0001 C CNN "LCSC"
 	1    9900 2900
 	0    -1   -1   0
@@
 F 2 "custom_parts:D_SOT-23_ANK" V 10800 2900 50  0001 C CNN
 F 3 "~" V 10800 2900 50  0001 C CNN
+F 4 "C2500" H 10800 2900 50  0001 C CNN "LCSC"
 	1    10800 2900
 	0    -1   -1   0
@@
 F 2 "custom_parts:D_SOT-23_ANK" V 11700 2900 50  0001 C CNN
 F 3 "~" V 11700 2900 50  0001 C CNN
+F 4 "C2500" H 11700 2900 50  0001 C CNN "LCSC"
 	1    11700 2900
 	0    -1   -1   0
@@
 F 2 "custom_parts:D_SOT-23_ANK" V 12600 2900 50  0001 C CNN
 F 3 "~" V 12600 2900 50  0001 C CNN
+F 4 "C2500" H 12600 2900 50  0001 C CNN "LCSC"
 	1    12600 2900
 	0    -1   -1   0
@@
 F 2 "custom_parts:D_SOT-23_ANK" V 7200 3550 50  0001 C CNN
 F 3 "~" V 7200 3550 50  0001 C CNN
+F 4 "C2500" H 7200 3550 50  0001 C CNN "LCSC"
 	1    7200 3550
 	0    -1   -1   0
@@
 F 2 "custom_parts:D_SOT-23_ANK" V 8100 3550 50  0001 C CNN
 F 3 "~" V 8100 3550 50  0001 C CNN
+F 4 "C2500" H 8100 3550 50  0001 C CNN "LCSC"
 	1    8100 3550
 	0    -1   -1   0
@@
 F 2 "custom_parts:D_SOT-23_ANK" V 9000 3550 50  0001 C CNN
 F 3 "~" V 9000 3550 50  0001 C CNN
+F 4 "C2500" H 9000 3550 50  0001 C CNN "LCSC"
 	1    9000 3550
 	0    -1   -1   0
@@
 F 2 "custom_parts:D_SOT-23_ANK" V 9900 3550 50  0001 C CNN
 F 3 "~" V 9900 3550 50  0001 C CNN
+F 4 "C2500" H 9900 3550 50  0001 C CNN "LCSC"
 	1    9900 3550
 	0    -1   -1   0
@@
 F 2 "custom_parts:D_SOT-23_ANK" V 10800 3550 50  0001 C CNN
 F 3 "~" V 10800 3550 50  0001 C CNN
+F 4 "C2500" H 10800 3550 50  0001 C CNN "LCSC"
 	1    10800 3550
 	0    -1   -1   0
@@
 F 2 "custom_parts:D_SOT-23_ANK" V 11700 3550 50  0001 C CNN
 F 3 "~" V 11700 3550 50  0001 C CNN
+F 4 "C2500" H 11700 3550 50  0001 C CNN "LCSC"
 	1    11700 3550
 	0    -1   -1   0
@@
 F 2 "custom_parts:D_SOT-23_ANK" V 12600 3550 50  0001 C CNN
 F 3 "~" V 12600 3550 50  0001 C CNN
+F 4 "C2500" H 12600 3550 50  0001 C CNN "LCSC"
 	1    12600 3550
 	0    -1   -1   0
@@
 F 2 "custom_parts:D_SOT-23_ANK" V 7200 4200 50  0001 C CNN
 F 3 "~" V 7200 4200 50  0001 C CNN
+F 4 "C2500" H 7200 4200 50  0001 C CNN "LCSC"
 	1    7200 4200
 	0    -1   -1   0
@@
 F 2 "custom_parts:D_SOT-23_ANK" V 8100 4200 50  0001 C CNN
 F 3 "~" V 8100 4200 50  0001 C CNN
+F 4 "C2500" H 8100 4200 50  0001 C CNN "LCSC"
 	1    8100 4200
 	0    -1   -1   0
@@
 F 2 "custom_parts:D_SOT-23_ANK" V 9000 4200 50  0001 C CNN
 F 3 "~" V 9000 4200 50  0001 C CNN
+F 4 "C2500" H 9000 4200 50  0001 C CNN "LCSC"
 	1    9000 4200
 	0    -1   -1   0
@@
 F 2 "custom_parts:D_SOT-23_ANK" V 9900 4200 50  0001 C CNN
 F 3 "~" V 9900 4200 50  0001 C CNN
+F 4 "C2500" H 9900 4200 50  0001 C CNN "LCSC"
 	1    9900 4200
 	0    -1   -1   0
@@
 F 2 "custom_parts:D_SOT-23_ANK" V 10800 4200 50  0001 C CNN
 F 3 "~" V 10800 4200 50  0001 C CNN
+F 4 "C2500" H 10800 4200 50  0001 C CNN "LCSC"
 	1    10800 4200
 	0    -1   -1   0
@@
 F 2 "custom_parts:D_SOT-23_ANK" V 11700 4200 50  0001 C CNN
 F 3 "~" V 11700 4200 50  0001 C CNN
+F 4 "C2500" H 11700 4200 50  0001 C CNN "LCSC"
 	1    11700 4200
 	0    -1   -1   0
@@
 F 2 "custom_parts:D_SOT-23_ANK" V 7200 4850 50  0001 C CNN
 F 3 "~" V 7200 4850 50  0001 C CNN
+F 4 "C2500" H 7200 4850 50  0001 C CNN "LCSC"
 	1    7200 4850
 	0    -1   -1   0
@@
 F 2 "custom_parts:D_SOT-23_ANK" V 8100 4850 50  0001 C CNN
 F 3 "~" V 8100 4850 50  0001 C CNN
+F 4 "C2500" H 8100 4850 50  0001 C CNN "LCSC"
 	1    8100 4850
 	0    -1   -1   0
@@
 F 2 "custom_parts:D_SOT-23_ANK" V 9000 4850 50  0001 C CNN
 F 3 "~" V 9000 4850 50  0001 C CNN
+F 4 "C2500" H 9000 4850 50  0001 C CNN "LCSC"
 	1    9000 4850
 	0    -1   -1   0
@@
 F 2 "custom_parts:D_SOT-23_ANK" V 9900 4850 50  0001 C CNN
 F 3 "~" V 9900 4850 50  0001 C CNN
+F 4 "C2500" H 9900 4850 50  0001 C CNN "LCSC"
 	1    9900 4850
 	0    -1   -1   0
@@
 F 2 "custom_parts:D_SOT-23_ANK" V 10800 4850 50  0001 C CNN
 F 3 "~" V 10800 4850 50  0001 C CNN
+F 4 "C2500" H 10800 4850 50  0001 C CNN "LCSC"
 	1    10800 4850
 	0    -1   -1   0
@@
 F 2 "custom_parts:D_SOT-23_ANK" V 11700 4850 50  0001 C CNN
 F 3 "~" V 11700 4850 50  0001 C CNN
+F 4 "C2500" H 11700 4850 50  0001 C CNN "LCSC"
 	1    11700 4850
 	0    -1   -1   0
@@
 F 2 "custom_parts:D_SOT-23_ANK" V 12600 4850 50  0001 C CNN
 F 3 "~" V 12600 4850 50  0001 C CNN
+F 4 "C2500" H 12600 4850 50  0001 C CNN "LCSC"
 	1    12600 4850
 	0    -1   -1   0
@@
 F 2 "custom_parts:D_SOT-23_ANK" V 7200 5500 50  0001 C CNN
 F 3 "~" V 7200 5500 50  0001 C CNN
+F 4 "C2500" H 7200 5500 50  0001 C CNN "LCSC"
 	1    7200 5500
 	0    -1   -1   0
@@
 F 2 "custom_parts:D_SOT-23_ANK" V 8100 5500 50  0001 C CNN
 F 3 "~" V 8100 5500 50  0001 C CNN
+F 4 "C2500" H 8100 5500 50  0001 C CNN "LCSC"
 	1    8100 5500
 	0    -1   -1   0
@@
 F 2 "Diode_SMD:D_SOD-123" V 11700 5500 50  0001 C CNN
 F 3 "~" V 11700 5500 50  0001 C CNN
+F 4 " C81598" H 11700 5500 50  0001 C CNN "LCSC"
 	1    11700 5500
 	0    -1   -1   0
@@
 F 2 "custom_parts:D_SOT-23_ANK" V 12600 5500 50  0001 C CNN
 F 3 "~" V 12600 5500 50  0001 C CNN
+F 4 "C2500" H 12600 5500 50  0001 C CNN "LCSC"
 	1    12600 5500
 	0    -1   -1   0
@@
 F 2 "custom_parts:D_SOT-23_ANK" V 13500 2900 50  0001 C CNN
 F 3 "~" V 13500 2900 50  0001 C CNN
+F 4 "C2500" H 13500 2900 50  0001 C CNN "LCSC"
 	1    13500 2900
 	0    -1   -1   0
@@
 F 2 "Diode_SMD:D_SOD-123" V 13500 3550 50  0001 C CNN
 F 3 "~" V 13500 3550 50  0001 C CNN
+F 4 " C81598" H 13500 3550 50  0001 C CNN "LCSC"
 	1    13500 3550
 	0    -1   -1   0
@@
 F 2 "custom_parts:D_SOT-23_ANK" V 13500 4200 50  0001 C CNN
 F 3 "~" V 13500 4200 50  0001 C CNN
+F 4 "C2500" H 13500 4200 50  0001 C CNN "LCSC"
 	1    13500 4200
 	0    -1   -1   0
@@
 F 2 "Diode_SMD:D_SOD-123" V 13500 4850 50  0001 C CNN
 F 3 "~" V 13500 4850 50  0001 C CNN
+F 4 " C81598" H 13500 4850 50  0001 C CNN "LCSC"
 	1    13500 4850
 	0    -1   -1   0
@@
 F 2 "custom_parts:D_SOT-23_ANK" V 13500 5500 50  0001 C CNN
 F 3 "~" V 13500 5500 50  0001 C CNN
+F 4 "C2500" H 13500 5500 50  0001 C CNN "LCSC"
 	1    13500 5500
 	0    -1   -1   0

Commit message: fix BOM
Parts:
- C7: LCSC C28323 -> C28323
- C8, C9: LCSC C1804 -> C1804
- D1, D10, D11, D12, D13, D14, D15, D17, D18, D19, D2, D20, D21, D22, D23, D24, D25, D26, D27, D28, D29, D3, D30, D32, D33, D35, D36, D4, D5, D6, D7, D8, D9: LCSC C2500 -> C8553
- D16, D31, D34: LCSC C81598 -> C81598
- RESET1: LCSC C318884 -> C318884
Changed lines of the file:
@@
 F 2 "Capacitor_SMD:C_0805_2012Metric" H 1950 8800 50  0001 C CNN
 F 3 "~" H 1950 8800 50  0001 C CNN
-F 4 " C28323" H 1950 8800 50  0001 C CNN "LCSC"
+F 4 "C28323" H 1950 8800 50  0001 C CNN "LCSC"
 	1    1950 8800
 	1    0    0    -1
@@
 F 2 "Capacitor_SMD:C_0805_2012Metric" H 1200 7500 50  0001 C CNN
 F 3 "~" H 1200 7500 50  0001 C CNN
-F 4 " C1804" V 1200 7500 50  0001 C CNN "LCSC"
+F 4 "C1804" V 1200 7500 50  0001 C CNN "LCSC"
 	1    1200 7500
 	0    1    1    0
@@
 F 2 "Capacitor_SMD:C_0805_2012Metric" H 1200 7850 50  0001 C CNN
 F 3 "~" H 1200 7850 50  0001 C CNN
-F 4 " C1804" V 1200 7850 50  0001 C CNN "LCSC"
+F 4 "C1804" V 1200 7850 50  0001 C CNN "LCSC"
 	1    1200 7850
 	0    1    1    0
@@
 F 2 "random-keyboard-parts:SKQG-1155865" H 2050 7450 50  0001 C CNN
 F 3 "~" H 2050 7450 50  0001 C CNN
-F 4 " C318884" H 2050 7250 50  0001 C CNN "LCSC"
+F 4 "C318884" H 2050 7250 50  0001 C CNN "LCSC"
 	1    2050 7250
 	1    0    0    -1
@@
 F 2 "custom_parts:D_SOT-23_ANK" V 7200 2900 50  0001 C CNN
 F 3 "~" V 7200 2900 50  0001 C CNN
-F 4 "C2500" H 7200 2900 50  0001 C CNN "LCSC"
+F 4 "C8553" H 7200 2900 50  0001 C CNN "LCSC"
 	1    7200 2900
 	0    -1   -1   0
@@
 F 2 "custom_parts:D_SOT-23_ANK" V 8100 2900 50  0001 C CNN
 F 3 "~" V 8100 2900 50  0001 C CNN
-F 4 "C2500" H 8100 2900 50  0001 C CNN "LCSC"
+F 4 "C8553" H 8100 2900 50  0001 C CNN "LCSC"
 	1    8100 2900
 	0    -1   -1   0
@@
 F 2 "custom_parts:D_SOT-23_ANK" V 9000 2900 50  0001 C CNN
 F 3 "~" V 9000 2900 50  0001 C CNN
-F 4 "C2500" H 9000 2900 50  0001 C CNN "LCSC"
+F 4 "C8553" H 9000 2900 50  0001 C CNN "LCSC"
 	1    9000 2900
 	0    -1   -1   0
@@
 F 2 "custom_parts:D_SOT-23_ANK" V 9900 2900 50  0001 C CNN
 F 3 "~" V 9900 2900 50  0001 C CNN
-F 4 "C2500" H 9900 2900 50  0001 C CNN "LCSC"
+F 4 "C8553" H 9900 2900 50  0001 C CNN "LCSC"
 	1    9900 2900
 	0    -1   -1   0
@@
 F 2 "custom_parts:D_SOT-23_ANK" V 10800 2900 50  0001 C CNN
 F 3 "~" V 10800 2900 50  0001 C CNN
-F 4 "C2500" H 10800 2900 50  0001 C CNN "LCSC"
+F 4 "C8553" H 10800 2900 50  0001 C CNN "LCSC"
 	1    10800 2900
 	0    -1   -1   0
@@
 F 2 "custom_parts:D_SOT-23_ANK" V 11700 2900 50  0001 C CNN
 F 3 "~" V 11700 2900 50  0001 C CNN
-F 4 "C2500" H 11700 2900 50  0001 C CNN "LCSC"
+F 4 "C8553" H 11700 2900 50  0001 C CNN "LCSC"
 	1    11700 2900
 	0    -1   -1   0
@@
 F 2 "custom_parts:D_SOT-23_ANK" V 12600 2900 50  0001 C CNN
 F 3 "~" V 12600 2900 50  0001 C CNN
-F 4 "C2500" H 12600 2900 50  0001 C CNN "LCSC"
+F 4 "C8553" H 12600 2900 50  0001 C CNN "LCSC"
 	1    12600 2900
 	0    -1   -1   0
@@
 F 2 "custom_parts:D_SOT-23_ANK" V 7200 3550 50  0001 C CNN
 F 3 "~" V 7200 3550 50  0001 C CNN
-F 4 "C2500" H 7200 3550 50  0001 C CNN "LCSC"
+F 4 "C8553" H 7200 3550 50  0001 C CNN "LCSC"
 	1    7200 3550
 	0    -1   -1   0
@@
 F 2 "custom_parts:D_SOT-23_ANK" V 8100 3550 50  0001 C CNN
 F 3 "~" V 8100 3550 50  0001 C CNN
-F 4 "C2500" H 8100 3550 50  0001 C CNN "LCSC"
+F 4 "C8553" H 8100 3550 50  0001 C CNN "LCSC"
 	1    8100 3550
 	0    -1   -1   0
@@
 F 2 "custom_parts:D_SOT-23_ANK" V 9000 3550 50  0001 C CNN
 F 3 "~" V 9000 3550 50  0001 C CNN
-F 4 "C2500" H 9000 3550 50  0001 C CNN "LCSC"
+F 4 "C8553" H 9000 3550 50  0001 C CNN "LCSC"
 	1    9000 3550
 	0    -1   -1   0
@@
 F 2 "custom_parts:D_SOT-23_ANK" V 9900 3550 50  0001 C CNN
 F 3 "~" V 9900 3550 50  0001 C CNN
-F 4 "C2500" H 9900 3550 50  0001 C CNN "LCSC"
+F 4 "C8553" H 9900 3550 50  0001 C CNN "LCSC"
 	1    9900 3550
 	0    -1   -1   0
@@
 F 2 "custom_parts:D_SOT-23_ANK" V 10800 3550 50  0001 C CNN
 F 3 "~" V 10800 3550 50  0001 C CNN
-F 4 "C2500" H 10800 3550 50  0001 C CNN "LCSC"
+F 4 "C8553" H 10800 3550 50  0001 C CNN "LCSC"
 	1    10800 3550
 	0    -1   -1   0
@@
 F 2 "custom_parts:D_SOT-23_ANK" V 11700 3550 50  0001 C CNN
 F 3 "~" V 11700 3550 50  0001 C CNN
-F 4 "C2500" H 11700 3550 50  0001 C CNN "LCSC"
+F 4 "C8553" H 11700 3550 50  0001 C CNN "LCSC"
 	1    11700 3550
 	0    -1   -1   0
@@
 F 2 "custom_parts:D_SOT-23_ANK" V 12600 3550 50  0001 C CNN
 F 3 "~" V 12600 3550 50  0001 C CNN
-F 4 "C2500" H 12600 3550 50  0001 C CNN "LCSC"
+F 4 "C8553" H 12600 3550 50  0001 C CNN "LCSC"
 	1    12600 3550
 	0    -1   -1   0
@@
 F 2 "custom_parts:D_SOT-23_ANK" V 7200 4200 50  0001 C CNN
 F 3 "~" V 7200 4200 50  0001 C CNN
-F 4 "C2500" H 7200 4200 50  0001 C CNN "LCSC"
+F 4 "C8553" H 7200 4200 50  0001 C CNN "LCSC"
 	1    7200 4200
 	0    -1   -1   0
@@
 F 2 "custom_parts:D_SOT-23_ANK" V 8100 4200 50  0001 C CNN
 F 3 "~" V 8100 4200 50  0001 C CNN
-F 4 "C2500" H 8100 4200 50  0001 C CNN "LCSC"
+F 4 "C8553" H 8100 4200 50  0001 C CNN "LCSC"
 	1    8100 4200
 	0    -1   -1   0
@@
 F 2 "custom_parts:D_SOT-23_ANK" V 9000 4200 50  0001 C CNN
 F 3 "~" V 9000 4200 50  0001 C CNN
-F 4 "C2500" H 9000 4200 50  0001 C CNN "LCSC"
+F 4 "C8553" H 9000 4200 50  0001 C CNN "LCSC"
 	1    9000 4200
 	0    -1   -1   0
@@
 F 2 "custom_parts:D_SOT-23_ANK" V 9900 4200 50  0001 C CNN
 F 3 "~" V 9900 4200 50  0001 C CNN
-F 4 "C2500" H 9900 4200 50  0001 C CNN "LCSC"
+F 4 "C8553" H 9900 4200 50  0001 C CNN "LCSC"
 	1    9900 4200
 	0    -1   -1   0
@@
 F 2 "custom_parts:D_SOT-23_ANK" V 10800 4200 50  0001 C CNN
 F 3 "~" V 10800 4200 50  0001 C CNN
-F 4 "C2500" H 10800 4200 50  0001 C CNN "LCSC"
+F 4 "C8553" H 10800 4200 50  0001 C CNN "LCSC"
 	1    10800 4200
 	0    -1   -1   0
@@
 F 2 "custom_parts:D_SOT-23_ANK" V 11700 4200 50  0001 C CNN
 F 3 "~" V 11700 4200 50  0001 C CNN
-F 4 "C2500" H 11700 4200 50  0001 C CNN "LCSC"
+F 4 "C8553" H 11700 4200 50  0001 C CNN "LCSC"
 	1    11700 4200
 	0    -1   -1   0
@@
 F 2 "custom_parts:D_SOT-23_ANK" V 7200 4850 50  0001 C CNN
 F 3 "~" V 7200 4850 50  0001 C CNN
-F 4 "C2500" H 7200 4850 50  0001 C CNN "LCSC"
+F 4 "C8553" H 7200 4850 50  0001 C CNN "LCSC"
 	1    7200 4850
 	0    -1   -1   0
@@
 F 2 "custom_parts:D_SOT-23_ANK" V 8100 4850 50  0001 C CNN
 F 3 "~" V 8100 4850 50  0001 C CNN
-F 4 "C2500" H 8100 4850 50  0001 C CNN "LCSC"
+F 4 "C8553" H 8100 4850 50  0001 C CNN "LCSC"
 	1    8100 4850
 	0    -1   -1   0
@@
 F 2 "custom_parts:D_SOT-23_ANK" V 9000 4850 50  0001 C CNN
 F 3 "~" V 9000 4850 50  0001 C CNN
-F 4 "C2500" H 9000 4850 50  0001 C CNN "LCSC"
+F 4 "C8553" H 9000 4850 50  0001 C CNN "LCSC"
 	1    9000 4850
 	0    -1   -1   0
@@
 F 2 "custom_parts:D_SOT-23_ANK" V 9900 4850 50  0001 C CNN
 F 3 "~" V 9900 4850 50  0001 C CNN
-F 4 "C2500" H 9900 4850 50  0001 C CNN "LCSC"
+F 4 "C8553" H 9900 4850 50  0001 C CNN "LCSC"
 	1    9900 4850
 	0    -1   -1   0
@@
 F 2 "custom_parts:D_SOT-23_ANK" V 10800 4850 50  0001 C CNN
 F 3 "~" V 10800 4850 50  0001 C CNN
-F 4 "C2500" H 10800 4850 50  0001 C CNN "LCSC"
+F 4 "C8553" H 10800 4850 50  0001 C CNN "LCSC"
 	1    10800 4850
 	0    -1   -1   0
@@
 F 2 "custom_parts:D_SOT-23_ANK" V 11700 4850 50  0001 C CNN
 F 3 "~" V 11700 4850 50  0001 C CNN
-F 4 "C2500" H 11700 4850 50  0001 C CNN "LCSC"
+F 4 "C8553" H 11700 4850 50  0001 C CNN "LCSC"
 	1    11700 4850
 	0    -1   -1   0
@@
 F 2 "custom_parts:D_SOT-23_ANK" V 12600 4850 50  0001 C CNN
 F 3 "~" V 12600 4850 50  0001 C CNN
-F 4 "C2500" H 12600 4850 50  0001 C CNN "LCSC"
+F 4 "C8553" H 12600 4850 50  0001 C CNN "LCSC"
 	1    12600 4850
 	0    -1   -1   0
@@
 F 2 "custom_parts:D_SOT-23_ANK" V 7200 5500 50  0001 C CNN
 F 3 "~" V 7200 5500 50  0001 C CNN
-F 4 "C2500" H 7200 5500 50  0001 C CNN "LCSC"
+F 4 "C8553" H 7200 5500 50  0001 C CNN "LCSC"
 	1    7200 5500
 	0    -1   -1   0
@@
 F 2 "custom_parts:D_SOT-23_ANK" V 8100 5500 50  0001 C CNN
 F 3 "~" V 8100 5500 50  0001 C CNN
-F 4 "C2500" H 8100 5500 50  0001 C CNN "LCSC"
+F 4 "C8553" H 8100 5500 50  0001 C CNN "LCSC"
 	1    8100 5500
 	0    -1   -1   0
@@
 F 2 "Diode_SMD:D_SOD-123" V 11700 5500 50  0001 C CNN
 F 3 "~" V 11700 5500 50  0001 C CNN
-F 4 " C81598" H 11700 5500 50  0001 C CNN "LCSC"
+F 4 "C81598" H 11700 5500 50  0001 C CNN "LCSC"
 	1    11700 5500
 	0    -1   -1   0
@@
 F 2 "custom_parts:D_SOT-23_ANK" V 12600 5500 50  0001 C CNN
 F 3 "~" V 12600 5500 50  0001 C CNN
-F 4 "C2500" H 12600 5500 50  0001 C CNN "LCSC"
+F 4 "C8553" H 12600 5500 50  0001 C CNN "LCSC"
 	1    12600 5500
 	0    -1   -1   0
@@
 F 2 "custom_parts:D_SOT-23_ANK" V 13500 2900 50  0001 C CNN
 F 3 "~" V 13500 2900 50  0001 C CNN
-F 4 "C2500" H 13500 2900 50  0001 C CNN "LCSC"
+F 4 "C8553" H 13500 2900 50  0001 C CNN "LCSC"
 	1    13500 2900
 	0    -1   -1   0
@@
 F 2 "Diode_SMD:D_SOD-123" V 13500 3550 50  0001 C CNN
 F 3 "~" V 13500 3550 50  0001 C CNN
-F 4 " C81598" H 13500 3550 50  0001 C CNN "LCSC"
+F 4 "C81598" H 13500 3550 50  0001 C CNN "LCSC"
 	1    13500 3550
 	0    -1   -1   0
@@
 F 2 "custom_parts:D_SOT-23_ANK" V 13500 4200 50  0001 C CNN
 F 3 "~" V 13500 4200 50  0001 C CNN
-F 4 "C2500" H 13500 4200 50  0001 C CNN "LCSC"
+F 4 "C8553" H 13500 4200 50  0001 C CNN "LCSC"
 	1    13500 4200
 	0    -1   -1   0
@@
 F 2 "Diode_SMD:D_SOD-123" V 13500 4850 50  0001 C CNN
 F 3 "~" V 13500 4850 50  0001 C CNN
-F 4 " C81598" H 13500 4850 50  0001 C CNN "LCSC"
+F 4 "C81598" H 13500 4850 50  0001 C CNN "LCSC"
 	1    13500 4850
 	0    -1   -1   0
@@
 F 2 "custom_parts:D_SOT-23_ANK" V 13500 5500 50  0001 C CNN
 F 3 "~" V 13500 5500 50  0001 C CNN
-F 4 "C2500" H 13500 5500 50  0001 C CNN "LCSC"
+F 4 "C8553" H 13500 5500 50  0001 C CNN "LCSC"
 	1    13500 5500
 	0    -1   -1   0
