File: noah.kicad_pcb (KiCad board)
At the start: 2 copper layers, 301.5 x 98.9 mm, 139 parts, among them U1 ATmega32U4-AU, U2 SRV05-4

Commit message: update BOM
Parts:
- renumbered RESET1 to RESET

Commit message: fix DB plug wire orientation
Parts:
- R4: value 470 -> 1k
- moved R2 2.55 mm to (264.0, 119.2)
- moved R1 2.53 mm to (261.4, 119.2)
- renumbered RESET to RESET1
Connections:
- U2 pad 1: D- -> D+
- U2 pad 4: D+ -> D-
- USB1 pad 2: D+ -> D-
- USB1 pad 3: D- -> D+
Routing:
- net Net-(R1-Pad2): track 142.1 -> 144.8 mm, vias 0 -> 2
- net Net-(R2-Pad2): track 141.7 -> 140.7 mm

Commit message: update gerbers
Parts:
- renumbered RESET1 to RESET
Changed lines of the file:
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@@
       (drillshape 0)
       (scaleselection 1)
-      (outputdirectory ""))
+      (outputdirectory "gerbers"))
   )
   (net 0 "")
@@
     (at 233.8705 168.2115)
     (attr smd)
-    (fp_text reference RESET1 (at 0 -4.064) (layer B.SilkS)
-      (effects (font (size 1 1) (thickness 0.15)) (justify mirror))
-    )
+    (fp_text reference RESET (at 0 -4.064) (layer B.SilkS)
+      (effects (font (size 1 1) (thickness 0.15)) (justify mirror))
+    )
